Commit message: updated

File: asbr_package/asbr_test_ws/install/asbr_description/share/asbr_description/urdf/asbr.urdf.xacro (robot description, xacro)
@@ -15,11 +15,8 @@
     <xacro:arg name="safety_k_position" default="20"/>
     <xacro:arg name="force_abs_paths" default="false"/>
-    <xacro:arg name="initial_positions_file" default="$(find ur_description)/config/initial_positions.yaml"/>
-    <!-- Load initial positions from YAML file -->
-    <xacro:property name="initial_positions" value="${xacro.load_yaml(initial_positions_file)['joint_positions']}"></xacro:property>
     <!-- Include the ur.urdf.xacro file -->
     <xacro:include filename="$(find ur_description)/urdf/ur.urdf.xacro"/>
     <!-- Include the Robotiq 2F-85 gripper -->
-    <xacro:include filename="$(find robotiq_2f_85_gripper_visualization)/urdf/robotiq_arg2f_85_model.xacro"/>
+    <xacro:include filename="$(find robotiq_description)/urdf/robotiq_arg2f_85_model.xacro"/>
     <!-- Connecting UR5e end-effector to gripper -->
     <joint name="end_effector_gripper_joint" type="fixed">
