Commit message: modification

File: asbr_package/asbr_test_ws/src/asbr_description/urdf/asbr.urdf.xacro (robot description, xacro)
@@ -15,4 +15,7 @@
     <xacro:arg name="safety_k_position" default="20"/>
     <xacro:arg name="force_abs_paths" default="false"/>
+    <xacro:arg name="initial_positions_file" default="$(find ur_description)/config/initial_positions.yaml"/>
+    <!-- Load initial positions from YAML file -->
+    <xacro:property name="initial_positions" value="${xacro.load_yaml(initial_positions_file)['joint_positions']}"></xacro:property>
     <!-- Include the ur.urdf.xacro file -->
     <xacro:include filename="$(find ur_description)/urdf/ur.urdf.xacro"/>

Commit message: modified the code since the initial joints to bringup UR5e is annoyingly not working

File: asbr_package/asbr_test_ws/src/asbr_description/urdf/asbr.urdf.xacro (robot description, xacro)
@@ -1,2 +1,3 @@
+ls
 <?xml version="1.0"?>
 <robot name="ur5e_robot" xmlns:xacro="http://www.ros.org/wiki/xacro">
@@ -15,7 +16,4 @@
     <xacro:arg name="safety_k_position" default="20"/>
     <xacro:arg name="force_abs_paths" default="false"/>
-    <xacro:arg name="initial_positions_file" default="$(find ur_description)/config/initial_positions.yaml"/>
-    <!-- Load initial positions from YAML file -->
-    <xacro:property name="initial_positions" value="${xacro.load_yaml(initial_positions_file)['joint_positions']}"></xacro:property>
     <!-- Include the ur.urdf.xacro file -->
     <xacro:include filename="$(find ur_description)/urdf/ur.urdf.xacro"/>

Commit message: added the camera based information from assignment2 asbr

File: asbr_package/asbr_test_ws/src/asbr_description/urdf/asbr.urdf.xacro (robot description, xacro)
@@ -15,8 +15,7 @@
     <xacro:arg name="safety_k_position" default="20"/>
     <xacro:arg name="force_abs_paths" default="false"/>
-    <!-- Include the ur.urdf.xacro file -->
     <xacro:include filename="$(find ur_description)/urdf/ur.urdf.xacro"/>
-    <!-- Include the Robotiq 2F-85 gripper -->
     <xacro:include filename="$(find robotiq_description)/urdf/robotiq_arg2f_85_model.xacro"/>
+    <xacro:include filename="$(find realsense2_description)/urdf/_d435.urdf.xacro"/>
     <!-- Connecting UR5e end-effector to gripper -->
     <joint name="end_effector_gripper_joint" type="fixed">
@@ -25,7 +24,16 @@
         <origin xyz="0 0 0" rpy="0 0 0"/>
     </joint>
-    <!-- Include the D435 sensor -->
-    <xacro:include filename="$(find realsense2_description)/urdf/_d435.urdf.xacro"/>
-    <!-- Connecting D435 to UR5e -->
-    <xacro:sensor_d435 parent="robotiq_arg2f_base_link" name="d435" origin="xyz='0 0 0.1' rpy='0 0 0'" use_nominal_extrinsics="true" add_plug="true" use_mesh="true"/>
+    <!-- Adding the intermediate link between the end effector and the sensor for potentially camera adapters-->
+    <link name="camera_link">
+    </link>
+    <joint name="camera_joint" type="fixed">
+        <axis xyz="0 0 1"/>
+        <origin xyz="-0.015 -0.05 0.015" rpy="0 0 0"/>
+        <parent link="tool0"/>
+        <child link="camera_link"/>
+    </joint>
+    <!-- Connecting the camera sensor to the camera link -->
+    <xacro:sensor_d435 parent="tool0" name="d435" use_nominal_extrinsics="true" add_plug="true" use_mesh="true"> <!-- The parent can also be camera_link -->
+        <origin xyz="0.0 -0.06 0.0" rpy="-1.5708 -1.5708 0"/>
+    </xacro:sensor_d435>
 </robot>

Commit message: Tried to add the adapter but my need some modifications later

File: asbr_package/asbr_test_ws/src/asbr_description/urdf/asbr.urdf.xacro (robot description, xacro)
@@ -15,10 +15,20 @@
     <xacro:arg name="safety_k_position" default="20"/>
     <xacro:arg name="force_abs_paths" default="false"/>
+    <!-- Necessary modules (macros) to use-->
     <xacro:include filename="$(find ur_description)/urdf/ur.urdf.xacro"/>
     <xacro:include filename="$(find robotiq_description)/urdf/robotiq_arg2f_85_model.xacro"/>
     <xacro:include filename="$(find realsense2_description)/urdf/_d435.urdf.xacro"/>
+    <xacro:include filename="$(find robotiq_description)/urdf/asbr_UR5e_adapter.xacro"/>
+    <!-- Using the adapter macro I seriously modified -->
+    <xacro:adapter prefix="UR5e_gripper"/>
+    <!-- Connecting the end-effector to the adapter firsr before the gripper -->
+     <joint name="end_effector_adapter_joint" type="fixed">
+        <parent link="tool0"/>
+        <child link="UR5e_gripper_adapter"/>
+        <origin xyz="0 0 0" rpy="0 0 0"></origin>
+     </joint>
     <!-- Connecting UR5e end-effector to gripper -->
-    <joint name="end_effector_gripper_joint" type="fixed">
-        <parent link="tool0"/>
+    <joint name="UR5e_adapter_gripper_joint" type="fixed">
+        <parent link="UR5e_gripper_adapter"/>
         <child link="robotiq_arg2f_base_link"/>
         <origin xyz="0 0 0" rpy="0 0 0"/>

Commit message: update to xacro and added launch file

File: asbr_package/asbr_test_ws/src/asbr_description/urdf/asbr.urdf.xacro (robot description, xacro)
@@ -1,50 +1,115 @@
 <?xml version="1.0"?>
 <robot name="ur5e_robot" xmlns:xacro="http://www.ros.org/wiki/xacro">
-    <!-- Developer: Seyi R. Afolayan -->
-    <!-- Arguments required by ur.urdf.xacro -->
-    <xacro:arg name="name" default="ur5e_robot"/>
-    <xacro:arg name="ur_type" default="ur5e"/>
-    <xacro:arg name="tf_prefix" default=""/>
-    <xacro:arg name="joint_limit_params" default="$(find ur_description)/config/ur5e/joint_limits.yaml"/>
-    <xacro:arg name="kinematics_params" default="$(find ur_description)/config/ur5e/default_kinematics.yaml"/>
-    <xacro:arg name="physical_params" default="$(find ur_description)/config/ur5e/physical_parameters.yaml"/>
-    <xacro:arg name="visual_params" default="$(find ur_description)/config/ur5e/visual_parameters.yaml"/>
-    <xacro:arg name="transmission_hw_interface" default=""/>
-    <xacro:arg name="safety_limits" default="false"/>
-    <xacro:arg name="safety_pos_margin" default="0.15"/>
-    <xacro:arg name="safety_k_position" default="20"/>
-    <xacro:arg name="force_abs_paths" default="false"/>
-    <!-- Necessary modules (macros) to use-->
-    <xacro:include filename="$(find asbr_description)/urdf/ur5e_ros2_control.xacro"></xacro:include>
-    <xacro:include filename="$(find ur_description)/urdf/ur.urdf.xacro"/>
-    <xacro:include filename="$(find robotiq_2f_85_gripper_visualization)/urdf/robotiq_arg2f_85_model.xacro"/>
-    <xacro:include filename="$(find realsense2_description)/urdf/_d435.urdf.xacro"/>
-    <xacro:include filename="$(find robotiq_2f_85_gripper_visualization)/urdf/asbr_UR5e_adapter.xacro"/>
-    <!-- Using the adapter macro I seriously modified -->
-    <xacro:adapter prefix="UR5e_gripper"/>
-    <!-- Connecting the end-effector to the adapter firsr before the gripper -->
-     <joint name="end_effector_adapter_joint" type="fixed">
-        <parent link="tool0"/>
-        <child link="UR5e_gripper_adapter"/>
-        <origin xyz="0 0 0" rpy="0 0 0"></origin>
-     </joint>
-    <!-- Connecting UR5e adapter to gripper -->
-    <joint name="UR5e_adapter_gripper_joint" type="fixed">
-        <parent link="UR5e_gripper_adapter"/>
-        <child link="robotiq_arg2f_base_link"/>
-        <origin xyz="0 0 0" rpy="0 0 0"/>
-    </joint>
-    <!-- Adding the intermediate link between the end effector and the sensor for potentially camera adapters-->
-    <link name="camera_link">
-    </link>
-    <joint name="camera_joint" type="fixed">
-        <axis xyz="0 0 1"/>
-        <origin xyz="-0.015 -0.05 0.015" rpy="0 0 0"/>
-        <parent link="tool0"/>
-        <child link="camera_link"/>
-    </joint>
-    <!-- Connecting the camera sensor to the camera link -->
-    <xacro:sensor_d435 parent="tool0" name="d435" use_nominal_extrinsics="true" add_plug="true" use_mesh="true"> <!-- The parent can also be camera_link -->
-        <origin xyz="0.0 -0.06 0.0" rpy="-1.5708 -1.5708 0"/>
-    </xacro:sensor_d435>
+  <!-- Developer:Seyi  R. Afolayan -->
+  <!-- Arguments required by ur.urdf.xacro -->
+  <!-- Necessary modules (macros) to use-->
+  <!--<xacro:include filename="$(find asbr_description)/urdf/ur5e_ros2_control.xacro"></xacro:include> -->
+  <xacro:include filename="$(find ur_description)/urdf/ur_macro.xacro"/>
+  <xacro:include filename="$(find robotiq_description)/urdf/robotiq_2f_85_macro.urdf.xacro"/>
+  <xacro:include filename="$(find robotiq_description)/urdf/ur_to_robotiq_adapter.urdf.xacro"/>
+  <xacro:include filename="$(find realsense2_description)/urdf/_d435.urdf.xacro"/>
+  <xacro:arg name="name" default="ur5e_robot"/>
+  <xacro:arg name="ur_type" default="ur5e"/>
+  <xacro:arg name="tf_prefix" default=""/>
+  <!-- parameters -->
+  <xacro:arg name="tf_prefix" default="" />
+  <xacro:arg name="joint_limit_params" default="$(find ur_description)/config/$(arg ur_type)/joint_limits.yaml"/>
+  <xacro:arg name="kinematics_params" default="$(find ur_description)/config/$(arg ur_type)/default_kinematics.yaml"/>
+  <xacro:arg name="physical_params" default="$(find ur_description)/config/$(arg ur_type)/physical_parameters.yaml"/>
+  <xacro:arg name="visual_params" default="$(find ur_description)/config/$(arg ur_type)/visual_parameters.yaml"/>
+  <xacro:arg name="transmission_hw_interface" default=""/>
+  <xacro:arg name="safety_limits" default="false"/>
+  <xacro:arg name="safety_pos_margin" default="0.15"/>
+  <xacro:arg name="safety_k_position" default="20"/>
+  <!-- ros2_control related parameters -->
+  <xacro:arg name="headless_mode" default="false" />
+  <xacro:arg name="robot_ip" default="0.0.0.0" />
+  <xacro:arg name="script_filename" default=""/>
+  <xacro:arg name="output_recipe_filename" default=""/>
+  <xacro:arg name="input_recipe_filename" default=""/>
+  <xacro:arg name="reverse_ip" default="0.0.0.0"/>
+  <xacro:arg name="script_command_port" default="50004"/>
+  <xacro:arg name="reverse_port" default="50001"/>
+  <xacro:arg name="script_sender_port" default="50002"/>
+  <xacro:arg name="trajectory_port" default="50003"/>
+  <!--   tool communication related parameters-->
+  <xacro:arg name="use_tool_communication" default="false" />
+  <xacro:arg name="tool_voltage" default="0" />
+  <xacro:arg name="tool_parity" default="0" />
+  <xacro:arg name="tool_baud_rate" default="115200" />
+  <xacro:arg name="tool_stop_bits" default="1" />
+  <xacro:arg name="tool_rx_idle_chars" default="1.5" />
+  <xacro:arg name="tool_tx_idle_chars" default="3.5" />
+  <xacro:arg name="tool_device_name" default="/tmp/ttyUR" />
+  <xacro:arg name="tool_tcp_port" default="54321" />
+  <!-- Simulation parameters -->
+  <xacro:arg name="use_fake_hardware" default="true" />
+  <xacro:arg name="fake_sensor_commands" default="false" />
+  <xacro:arg name="sim_gazebo" default="false" />
+  <xacro:arg name="sim_ignition" default="false" />
+  <xacro:arg name="simulation_controllers" default="" />
+  <!-- initial position for simulations (Fake Hardware, Gazebo, Ignition) -->
+  <xacro:arg name="initial_positions_file" default="$(find ur_description)/config/initial_positions.yaml"/>
+  <!-- convert to property to use substitution in function -->
+  <xacro:property name="initial_positions_file" default="$(arg initial_positions_file)"/>
+  <!-- create link fixed to the "world" -->
+  <link name="world" />
+  <!-- UR5e -->
+  <xacro:ur_robot
+      name="$(arg name)"
+      tf_prefix="$(arg tf_prefix)"
+      parent="world"
+      joint_limits_parameters_file="$(arg joint_limit_params)"
+      kinematics_parameters_file="$(arg kinematics_params)"
+      physical_parameters_file="$(arg physical_params)"
+      visual_parameters_file="$(arg visual_params)"
+      transmission_hw_interface="$(arg transmission_hw_interface)"
+      safety_limits="$(arg safety_limits)"
+      safety_pos_margin="$(arg safety_pos_margin)"
+      safety_k_position="$(arg safety_k_position)"
+      use_fake_hardware="$(arg use_fake_hardware)"
+      fake_sensor_commands="$(arg fake_sensor_commands)"
+      sim_gazebo="$(arg sim_gazebo)"
+      sim_ignition="$(arg sim_ignition)"
+      headless_mode="$(arg headless_mode)"
+      initial_positions="${xacro.load_yaml(initial_positions_file)}"
+      use_tool_communication="$(arg use_tool_communication)"
+      tool_voltage="$(arg tool_voltage)"
+      tool_parity="$(arg tool_parity)"
+      tool_baud_rate="$(arg tool_baud_rate)"
+      tool_stop_bits="$(arg tool_stop_bits)"
+      tool_rx_idle_chars="$(arg tool_rx_idle_chars)"
+      tool_tx_idle_chars="$(arg tool_tx_idle_chars)"
+      tool_device_name="$(arg tool_device_name)"
+      tool_tcp_port="$(arg tool_tcp_port)"
+      robot_ip="$(arg robot_ip)"
+      script_filename="$(arg script_filename)"
+      output_recipe_filename="$(arg output_recipe_filename)"
+      input_recipe_filename="$(arg input_recipe_filename)"
+      reverse_ip="$(arg reverse_ip)"
+      script_command_port="$(arg script_command_port)"
+      reverse_port="$(arg reverse_port)"
+      script_sender_port="$(arg script_sender_port)"
+      trajectory_port="$(arg trajectory_port)"
+      >
+    <origin xyz="0 0 0" rpy="0 0 0" />          <!-- position robot in the world -->
+  </xacro:ur_robot>
+  <!-- UR to Robotiq adapter -->
+  <xacro:ur_to_robotiq prefix="" connected_to="tool0" />
+  <xacro:robotiq_gripper name="gripper" prefix="" parent="gripper_mount_link" use_fake_hardware="$(arg use_fake_hardware)">
+    <origin xyz="0 0 0" rpy="0 0 0" />
+  </xacro:robotiq_gripper>
+  <!-- Adding the intermediate link between the end effector and the sensor for potentially camera adapters-->
+  <link name="camera_link">
+  </link>
+  <joint name="camera_joint" type="fixed">
+    <axis xyz="0 0 1"/>
+    <origin xyz="-0.015 -0.05 0.015" rpy="0 0 0"/>
+    <parent link="tool0"/>
+    <child link="camera_link"/>
+  </joint>
+  <!-- Connecting the camera sensor to the camera link -->
+  <xacro:sensor_d435 parent="tool0" name="d435" use_nominal_extrinsics="true" add_plug="true" use_mesh="true">
+    <origin xyz="0.0 -0.06 0.0" rpy="-1.5708 -1.5708 0"/>
+  </xacro:sensor_d435>
 </robot>

File: asbr_package/asbr_test_ws/src/asbr_description/urdf/ur5e_ros2_control.xacro (robot description, xacro)
@@ -1,5 +1,5 @@
 <?xml version="1.0"?>
 <robot name="ur5e_robot" xmlns:xacro="http://www.ros.org/wiki/xacro">
-    <!-- Developer: Seyi R. Afolayan -->
+    <!-- Developer:Seyi R. Afolayan -->
     <!-- Adding the ros2_control tags for the UR5e cobot - The hardware interface for the controller manager-->
     <ros2_control name="GazeboSystem" type="system">
